Commit message: Updated finger joints to mimick parent joint

File: install/robotic_hand_description/share/robotic_hand_description/urdf/robotic_hand.urdf.xacro (robot description, xacro)
@@ -73,5 +73,5 @@
                                 xyz="${Index_length / 2.0} 0 0" rpy="0 ${pi / 2.0} 0" />
         </link>
-        <joint name="base_Index1_joint" type="revolute">
+        <joint name="Index_finger" type="revolute">
             <parent link="base_link" />
             <child link="Index1_link" />
@@ -103,4 +103,5 @@
             <axis xyz="0 1 0" />
             <limit lower="0" upper="-1.57" effort="100" velocity="100" />
+            <mimic joint="Index_finger" multiplier="1.0" offset="0.0"/>
         </joint>
         <link name="Index3_link">
@@ -127,4 +128,5 @@
             <axis xyz="0 1 0" />
             <limit lower="0" upper="-1.57" effort="100" velocity="100" />
+            <mimic joint="Index_finger" multiplier="1.0" offset="0.0"/>
         </joint>
 <!-- Middle Finger -->
@@ -146,5 +148,5 @@
                                 xyz="${Middle_length / 2.0} 0 0" rpy="0 ${pi / 2.0} 0" />
         </link>
-        <joint name="base_Middle1_joint" type="revolute">
+        <joint name="Middle_finger" type="revolute">
             <parent link="base_link" />
             <child link="Middle1_link" />
@@ -176,4 +178,5 @@
             <axis xyz="0 1 0" />
             <limit lower="0" upper="-1.57" effort="100" velocity="100" />
+            <mimic joint="Middle_finger" multiplier="1.0" offset="0.0"/>
         </joint>
         <link name="Middle3_link">
@@ -200,4 +203,5 @@
             <axis xyz="0 1 0" />
             <limit lower="0" upper="-1.57" effort="100" velocity="100" />
+            <mimic joint="Middle_finger" multiplier="1.0" offset="0.0"/>
         </joint>
 <!-- Ring Finger -->
@@ -219,5 +223,5 @@
                                 xyz="${Ring_length / 2.0} 0 0" rpy="0 ${pi / 2.0} 0" />
         </link>
-        <joint name="base_Ring1_joint" type="revolute">
+        <joint name="Ring_finger" type="revolute">
             <parent link="base_link" />
             <child link="Ring1_link" />
@@ -249,4 +253,5 @@
             <axis xyz="0 1 0" />
             <limit lower="0" upper="-1.57" effort="100" velocity="100" />
+            <mimic joint="Ring_finger" multiplier="1.0" offset="0.0"/>
         </joint>
         <link name="Ring3_link">
@@ -273,4 +278,5 @@
             <axis xyz="0 1 0" />
             <limit lower="0" upper="-1.57" effort="100" velocity="100" />
+            <mimic joint="Ring_finger" multiplier="1.0" offset="0.0"/>
         </joint>
 <!-- Pinky Finger -->
@@ -292,5 +298,5 @@
                                 xyz="${Pinky_length / 2.0} 0 0" rpy="0 ${pi / 2.0} 0" />
         </link>
-        <joint name="base_Pinky1_joint" type="revolute">
+        <joint name="Pinky_finger" type="revolute">
             <parent link="base_link" />
             <child link="Pinky1_link" />
@@ -322,4 +328,5 @@
             <axis xyz="0 1 0" />
             <limit lower="0" upper="-1.57" effort="100" velocity="100" />
+            <mimic joint="Pinky_finger" multiplier="1.0" offset="0.0"/>
         </joint>
         <link name="Pinky3_link">
@@ -346,4 +353,5 @@
             <axis xyz="0 1 0" />
             <limit lower="0" upper="-1.57" effort="100" velocity="100" />
+            <mimic joint="Pinky_finger" multiplier="1.0" offset="0.0"/>
         </joint>
         <!-- Thumb Finger-->
@@ -365,5 +373,5 @@
                                 xyz="0 ${-Thumb_length / 2.0} 0" rpy="${pi / 2.0} 0 0" />
         </link>
-        <joint name="base_Thumb1_joint" type="revolute">
+        <joint name="Thumb" type="revolute">
             <parent link="base_link" />
             <child link="Thumb1_link" />
@@ -395,4 +403,5 @@
             <axis xyz="1 0 0" />
             <limit lower="0" upper="-1.57" effort="100" velocity="100" />
+            <mimic joint="Thumb" multiplier="1.0" offset="0.0"/>
         </joint>
 </robot>

Commit message: Normalized coordinates to -0.785 from -1.57 which was causing fingers to intersect with palm

File: install/robotic_hand_description/share/robotic_hand_description/urdf/robotic_hand.urdf.xacro (robot description, xacro)
@@ -78,5 +78,5 @@
             <origin xyz="${base_length / 2} -0.11 0" rpy="0 0 0" />
             <axis xyz="0 1 0" />
-            <limit lower="0" upper="-1.57" effort="100" velocity="100" />
+            <limit lower="0" upper="-0.785" effort="100" velocity="100" />
         </joint>
         <link name="Index2_link">
@@ -102,5 +102,5 @@
             <origin xyz="${Index_length} 0 0" rpy="0 0 0" />
             <axis xyz="0 1 0" />
-            <limit lower="0" upper="-1.57" effort="100" velocity="100" />
+            <limit lower="0" upper="-0.785" effort="100" velocity="100" />
             <mimic joint="Index_finger" multiplier="1.0" offset="0.0"/>
         </joint>
@@ -127,5 +127,5 @@
             <origin xyz="${Index_length} 0 0" rpy="0 0 0" />
             <axis xyz="0 1 0" />
-            <limit lower="0" upper="-1.57" effort="100" velocity="100" />
+            <limit lower="0" upper="-0.785" effort="100" velocity="100" />
             <mimic joint="Index_finger" multiplier="1.0" offset="0.0"/>
         </joint>
@@ -153,5 +153,5 @@
             <origin xyz="${base_length / 2.0} -0.06 0" rpy="0 0 0" />
             <axis xyz="0 1 0" />
-            <limit lower="0" upper="-1.57" effort="100" velocity="100" />
+            <limit lower="0" upper="-0.785" effort="100" velocity="100" />
         </joint>
         <link name="Middle2_link">
@@ -177,5 +177,5 @@
             <origin xyz="${Middle_length} 0 0" rpy="0 0 0" />
             <axis xyz="0 1 0" />
-            <limit lower="0" upper="-1.57" effort="100" velocity="100" />
+            <limit lower="0" upper="-0.785" effort="100" velocity="100" />
             <mimic joint="Middle_finger" multiplier="1.0" offset="0.0"/>
         </joint>
@@ -202,5 +202,5 @@
             <origin xyz="${Middle_length} 0 0" rpy="0 0 0" />
             <axis xyz="0 1 0" />
-            <limit lower="0" upper="-1.57" effort="100" velocity="100" />
+            <limit lower="0" upper="-0.785" effort="100" velocity="100" />
             <mimic joint="Middle_finger" multiplier="1.0" offset="0.0"/>
         </joint>
@@ -228,5 +228,5 @@
             <origin xyz="${base_length / 2.0} 0 0" rpy="0 0 0" />
             <axis xyz="0 1 0" />
-            <limit lower="0" upper="-1.57" effort="100" velocity="100" />
+            <limit lower="0" upper="-0.785" effort="100" velocity="100" />
         </joint>
         <link name="Ring2_link">
@@ -252,5 +252,5 @@
             <origin xyz="${Ring_length} 0 0" rpy="0 0 0" />
             <axis xyz="0 1 0" />
-            <limit lower="0" upper="-1.57" effort="100" velocity="100" />
+            <limit lower="0" upper="-0.785" effort="100" velocity="100" />
             <mimic joint="Ring_finger" multiplier="1.0" offset="0.0"/>
         </joint>
@@ -277,5 +277,5 @@
             <origin xyz="${Ring_length} 0 0" rpy="0 0 0" />
             <axis xyz="0 1 0" />
-            <limit lower="0" upper="-1.57" effort="100" velocity="100" />
+            <limit lower="0" upper="-0.785" effort="100" velocity="100" />
             <mimic joint="Ring_finger" multiplier="1.0" offset="0.0"/>
         </joint>
@@ -303,5 +303,5 @@
             <origin xyz="${base_length / 2.0} 0.06 0" rpy="0 0 0" />
             <axis xyz="0 1 0" />
-            <limit lower="0" upper="-1.57" effort="100" velocity="100" />
+            <limit lower="0" upper="-0.785" effort="100" velocity="100" />
         </joint>
         <link name="Pinky2_link">
@@ -327,5 +327,5 @@
             <origin xyz="${Pinky_length} 0 0" rpy="0 0 0" />
             <axis xyz="0 1 0" />
-            <limit lower="0" upper="-1.57" effort="100" velocity="100" />
+            <limit lower="0" upper="-0.785" effort="100" velocity="100" />
             <mimic joint="Pinky_finger" multiplier="1.0" offset="0.0"/>
         </joint>
@@ -352,5 +352,5 @@
             <origin xyz="${Pinky_length} 0 0" rpy="0 0 0" />
             <axis xyz="0 1 0" />
-            <limit lower="0" upper="-1.57" effort="100" velocity="100" />
+            <limit lower="0" upper="-0.785" effort="100" velocity="100" />
             <mimic joint="Pinky_finger" multiplier="1.0" offset="0.0"/>
         </joint>
@@ -378,5 +378,5 @@
             <origin xyz="0 ${-base_width /2.0} 0" rpy="0 0 0" />
             <axis xyz="1 0 0" />
-            <limit lower="0" upper="-1.57" effort="100" velocity="100" />
+            <limit lower="0" upper="-0.785" effort="100" velocity="100" />
         </joint>
         <link name="Thumb2_link">
@@ -402,5 +402,5 @@
             <origin xyz="0 ${-Thumb_length} 0" rpy="0 0 0" />
             <axis xyz="1 0 0" />
-            <limit lower="0" upper="-1.57" effort="100" velocity="100" />
+            <limit lower="0" upper="-0.785" effort="100" velocity="100" />
             <mimic joint="Thumb" multiplier="1.0" offset="0.0"/>
         </joint>
